File: Board/micropet_v1.brd (EAGLE design)
At the start: 160 x 100 mm, 83 parts, among them IC1 LM317, IC10 PIAPLCC, IC11 PIAPLCC, IC12 7417N, IC13 RAMSOCK32TO512K, IC14 ROMSOCK32TO512K, IC3 74HCT00N, IC4 74LS86N, IC5 74LS145N, IC6 MC3446, IC7 MC3446, IC8 MC3446, IC9 VIAPLCC, P1 C64KEYB, P2 IEEE488, P3 PETUSERPORT, P5 CBMTAPE, P6 CBMTAPE, P7 PETKEYBD

Commit message: Board Rev 1.0F
Connections:
- net GND: no longer QG1.1
Routing:
- net GND: track 955.3 -> 935.9 mm
Other:
- board text added: "MicroPET-V1.0F"
- board text removed: "MicroPET-V1.0E"
Changed lines of the file:
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@@
 <wire x1="159.37" y1="99.53" x2="-0.63" y2="99.53" width="0" layer="20"/>
 <wire x1="-0.63" y1="99.53" x2="-0.63" y2="-0.47" width="0" layer="20"/>
-<text x="4.445" y="20.6375" size="1.778" layer="1" font="vector" rot="R90">MicroPET-V1.0E</text>
+<text x="4.445" y="20.6375" size="1.778" layer="1" font="vector" rot="R90">MicroPET-V1.0F</text>
 <text x="4.28625" y="58.499375" size="1.778" layer="1" font="vector" rot="R90">(C) 2020 A. Fachat</text>
-<text x="4.445" y="20.6375" size="1.778" layer="25" font="vector" rot="R90">MicroPET-V1.0E</text>
+<text x="4.445" y="20.6375" size="1.778" layer="25" font="vector" rot="R90">MicroPET-V1.0F</text>
 <text x="4.28625" y="58.499375" size="1.778" layer="25" font="vector" rot="R90">(C) 2020 A. Fachat</text>
 </plain>
@@
 <contactref element="IC14" pad="16"/>
 <contactref element="QG1" pad="7"/>
-<contactref element="QG1" pad="1"/>
 <contactref element="C14" pad="1"/>
 <contactref element="C16" pad="-"/>
@@
 <wire x1="38.57625" y1="18.57375" x2="40.48125" y2="18.57375" width="0.3048" layer="1"/>
 <wire x1="40.48125" y1="18.57375" x2="43.02125" y2="21.11375" width="0.3048" layer="1"/>
-<wire x1="61.9125" y1="23.65375" x2="61.9125" y2="18.7325" width="0.3048" layer="1"/>
-<wire x1="61.9125" y1="18.7325" x2="61.9125" y2="3.4925" width="0.3048" layer="1"/>
 <wire x1="57.15" y1="2.54" x2="60.96" y2="2.54" width="0.3048" layer="1"/>
 <wire x1="60.96" y1="2.54" x2="61.9125" y2="3.4925" width="0.3048" layer="1"/>
@@
 <wire x1="53.63875" y1="19.70375" x2="53.6575" y2="18.415" width="1.016" layer="1"/>
 <wire x1="53.6575" y1="18.415" x2="57.4675" y2="18.415" width="1.016" layer="16"/>
-<wire x1="57.4675" y1="18.415" x2="61.595" y2="18.415" width="0.3048" layer="16"/>
-<wire x1="61.595" y1="18.415" x2="61.9125" y2="18.7325" width="0.3048" layer="16"/>
 <wire x1="58.26125" y1="70.1675" x2="57.62625" y2="70.1675" width="0.3048" layer="16"/>
 <wire x1="57.62625" y1="70.1675" x2="56.35625" y2="68.8975" width="0.3048" layer="16"/>
@@
 <wire x1="57.4675" y1="49.450625" x2="55.800625" y2="49.450625" width="0.3048" layer="16"/>
 <wire x1="55.800625" y1="49.450625" x2="55.5625" y2="49.68875" width="0.3048" layer="16"/>
+<wire x1="57.4675" y1="18.415" x2="57.4675" y2="20.47875" width="0.3048" layer="1"/>
+<wire x1="57.4675" y1="20.47875" x2="58.499375" y2="21.510625" width="0.3048" layer="1"/>
+<wire x1="58.499375" y1="21.510625" x2="58.499375" y2="23.1775" width="0.3048" layer="1"/>
+<wire x1="58.499375" y1="23.1775" x2="58.42" y2="23.256875" width="0.3048" layer="1"/>
 </signal>
 <signal name="VCC">

Commit message: Board Rev 1.1A
Parts:
- removed IC14: ROMSOCK32TO512K, csa:DIL32OPT28
- added U$4: SPIFLASH, csa:DIL08
Connections:
- removed net /PGM: IC14.31, U$2.17
- removed net /ROMSEL: IC14.22, IC14.24, U$2.19
- removed net RA12: IC14.4, U$2.9
- removed net RA13: IC14.28, U$2.10
- removed net RA14: IC14.29, U$2.11
- removed net RA15: IC14.3, U$2.12
- removed net RA16: IC14.2, U$2.13
- removed net RA17: IC14.30, U$2.14
- removed net RA18: IC14.1, U$2.15
- new net N$11: U$2.15, U$4.1
- new net N$12: U$2.14, U$4.6
- new net N$13: U$2.13, U$4.2
- new net N$14: U$2.11, U$4.5
- net A0: no longer IC14.12
- net A1: no longer IC14.11
- net A10: no longer IC14.23
- net A11: no longer IC14.25
- net A2: no longer IC14.10
- net A3: no longer IC14.9
- net A4: no longer IC14.8
- net A5: no longer IC14.7
- net A6: no longer IC14.6
- net A7: no longer IC14.5
- net A8: no longer IC14.27
- net A9: no longer IC14.26
- net D0: no longer IC14.13
- net D1: no longer IC14.14
- net D2: no longer IC14.15
- net D3: no longer IC14.17
- net D4: no longer IC14.18
- net D5: no longer IC14.19
- net D6: no longer IC14.20
- net D7: no longer IC14.21
- net GND: now also U$4.4; no longer IC14.16
- net VCMOS: now also U$4.7, U$4.8; no longer IC14.32
Routing:
- net RA18: track 96.9 -> 0.00 mm, vias 1 -> 0
- net RA17: track 94.2 -> 0.00 mm, vias 2 -> 0
- net RA14: track 93.9 -> 0.00 mm, vias 2 -> 0
- net RA13: track 90.9 -> 0.00 mm, vias 2 -> 0
- net RA16: track 88.6 -> 0.00 mm, vias 1 -> 0
- net RA15: track 85.7 -> 0.00 mm, vias 1 -> 0
- net /PGM: track 81.8 -> 0.00 mm, vias 1 -> 0
- net RA12: track 80.2 -> 0.00 mm, vias 1 -> 0
- net /ROMSEL: track 62.1 -> 0.00 mm, vias 1 -> 0
- net N$11: track 0.00 -> 59.9 mm, vias 0 -> 2
- net N$13: track 0.00 -> 53.0 mm, vias 0 -> 2
- net A7: track 66.7 -> 14.6 mm, vias 2 -> 0
- net N$12: track 0.00 -> 46.1 mm, vias 0 -> 2
- net D2: track 176.1 -> 131.6 mm, vias 8 -> 6
- net VCMOS: track 578.2 -> 535.8 mm, vias 15 -> 13
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Other:
- board text added: "MicroPET-V1.1A"
- board text removed: "MicroPET-V1.0F"

Commit message: Board version 1.1B
Parts:
- removed JP8: (no value), jumper:JP2
Connections:
- removed net MODE1: JP8.2, U$2.58
- new net PHI2_IO: IC10.28, IC11.28, IC9.27, U$2.58
- net GND: no longer JP8.1
- net PHI2: no longer IC10.28, IC11.28, IC9.27
- net V33: no longer JP8.3
Routing:
- net PHI2_IO: track 0.00 -> 137.8 mm, vias 0 -> 6
- net PHI2: track 168.5 -> 87.8 mm, vias 6 -> 4
- net MODE1: track 27.7 -> 0.00 mm, vias 2 -> 0
- net GND: track 911.2 -> 902.1 mm
- net V33: track 193.1 -> 189.1 mm
- net VPA: track 59.7 -> 58.1 mm
Other:
- board text added: "(C) 2020,2021 A. Fachat"
- board text added: "MicroPET-V1.1B"
- board text removed: "(C) 2020 A. Fachat"
- board text removed: "MicroPET-V1.1A"
