File: Board/micropet_v1.sch (EAGLE design)
At the start: 83 parts, among them IC1 LM317, IC10 PIAPLCC, IC11 PIAPLCC, IC12 7417N, IC13 RAMSOCK32TO512K, IC14 ROMSOCK32TO512K, IC3 74HCT00N, IC4 74LS86N, IC5 74LS145N, IC6 MC3446, IC7 MC3446, IC8 MC3446, IC9 VIAPLCC, P1 C64KEYB, P2 IEEE488, P3 PETUSERPORT, P5 CBMTAPE, P6 CBMTAPE, P7 PETKEYBD

Commit message: Board Rev 1.0F
Connections:
- net GND: no longer QG1.CON
Other:
- note added: "1.0F: don't pull CON pin of the clock oscillator to gnd (disables oscillators with Tri-state input)"
- note added: "MICROPET-V1.0F"
- note added: "MICROPET-V1.0F-20201228"
- note added: "TODO: Connect CPU E and VPB to CPLD"
Changed lines of the file:
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@@
 <part name="QG1" library="crystal" deviceset="CRYSTAL_RES-" device="SG51"/>
 <part name="GND10" library="supply1" deviceset="GND" device=""/>
-<part name="GND12" library="supply1" deviceset="GND" device=""/>
 <part name="SUPPLY2" library="supply2" deviceset="VCC" device=""/>
 <part name="IC1" library="v-reg" deviceset="LM317TL" device="" value="LM317"/>
@@
 <description>RAM,ROM,CPU</description>
 <plain>
-<text x="271.78" y="0" size="2.54" layer="92">MICROPET-V1.0E-20201224</text>
-<text x="271.78" y="22.86" size="3.81" layer="92">MICROPET-V1.0E</text>
+<text x="271.78" y="0" size="2.54" layer="92">MICROPET-V1.0F-20201228</text>
+<text x="271.78" y="22.86" size="3.81" layer="92">MICROPET-V1.0F</text>
 <text x="271.78" y="17.78" size="2.54" layer="92">(C) A. Fachat</text>
 <text x="337.82" y="20.32" size="2.54" layer="92">SHEET 2/3</text>
@@
 <text x="279.4" y="43.18" size="2.54" layer="94">1.0D: pull up resistor on Phi2 to improve phi2 signal quality</text>
 <text x="279.4" y="48.26" size="2.54" layer="94">1.0E: Add bypass caps to V33 (3.3V CPLD power supply)</text>
+<text x="279.4" y="73.66" size="2.54" layer="94">TODO: Connect CPU E and VPB to CPLD</text>
+<text x="279.4" y="53.34" size="2.54" layer="94">1.0F: don't pull CON pin of the clock oscillator to gnd
+         (disables oscillators with Tri-state input)</text>
 </plain>
 <instances>
@@
 <instance part="QG1" gate="A" x="81.28" y="190.5"/>
 <instance part="GND10" gate="1" x="66.04" y="177.8"/>
-<instance part="GND12" gate="1" x="101.6" y="193.04"/>
 <instance part="SUPPLY2" gate="G$1" x="66.04" y="200.66"/>
 <instance part="IC14" gate="G$2" x="0" y="5.08"/>
@@
 </segment>
 <segment>
-<pinref part="QG1" gate="A" pin="CON"/>
-<pinref part="GND12" gate="1" pin="GND"/>
-<wire x1="93.98" y1="195.58" x2="101.6" y2="195.58" width="0.1524" layer="91"/>
-</segment>
-<segment>

Commit message: Board Rev 1.1A
Parts:
- removed IC14: ROMSOCK32TO512K, csa:ROMSOCK32TO512K
- added U$4: SPIFLASH, csa:SPIFLASH
Connections:
- removed net /PGM: IC14G$1./PGM, U$2G$3.FB2MC15
- removed net /ROMSEL: IC14G$1./CE, IC14G$1./OE, U$2G$3.FB2MC17
- removed net RA12: IC14G$1.A12, U$2G$3.FB2MC2
- removed net RA13: IC14G$1.A13, U$2G$3.FB2MC3
- removed net RA14: IC14G$1.A14, U$2G$3.FB2MC5
- removed net RA15: IC14G$1.A15/VPP, U$2G$3.FB2MC6
- removed net RA16: IC14G$1.A16, U$2G$3.FB2MC8
- removed net RA17: IC14G$1.A17/VCC, U$2G$3.FB2MC10
- removed net RA18: IC14G$1.A18/VPP, U$2G$3.FB2MC12
- new net N$11: U$2G$3.FB2MC12, U$4./CS
- new net N$12: U$2G$3.FB2MC10, U$4.SCK
- new net N$13: U$2G$3.FB2MC8, U$4.SO
- new net N$14: U$2G$3.FB2MC5, U$4.SI
- net A0: no longer IC14G$1.A0
- net A1: no longer IC14G$1.A1
- net A10: no longer IC14G$1.A10
- net A11: no longer IC14G$1.A11
- net A2: no longer IC14G$1.A2
- net A3: no longer IC14G$1.A3
- net A4: no longer IC14G$1.A4
- net A5: no longer IC14G$1.A5
- net A6: no longer IC14G$1.A6
- net A7: no longer IC14G$1.A7
- net A8: no longer IC14G$1.A8
- net A9: no longer IC14G$1.A9
- net D0: no longer IC14G$1.O0
- net D1: no longer IC14G$1.O1
- net D2: no longer IC14G$1.O2
- net D3: no longer IC14G$1.O3
- net D4: no longer IC14G$1.O4
- net D5: no longer IC14G$1.O5
- net D6: no longer IC14G$1.O6
- net D7: no longer IC14G$1.O7
- net GND: now also U$4.GND; no longer IC14G$2.GND
- net VCMOS: now also U$4./HOLD, U$4.VCC; no longer IC14G$2.VCC
Other:
- note added: "1.1A: replace parallel ROM with SPI Flash"
- note added: "MICROPET-V1.0F-20210106"
- note added: "MICROPET-V1.1A"
- note added: "MICROPET-V1.1A-20210106"
- note added: "MICROPET-V1.1A-20210601"
- note removed: "MICROPET-V1.0A-20200705"
- note removed: "MICROPET-V1.0E"
- note removed: "MICROPET-V1.0E-20201224"
- note removed: "MICROPET-V1.0F"
- note removed: "MICROPET-V1.0F-20201228"

Commit message: Board version 1.1B
Parts:
- removed JP8: (no value), jumper:JP2E
Connections:
- removed net MODE1: JP8.2, U$2G$3.FB9MC14
- new net PHI2_IO: IC10G$1.PHI2, IC11G$1.PHI2, IC9G$1.PHI2, U$2G$3.FB9MC14
- net GND: no longer JP8.1
- net PHI2: no longer IC10G$1.PHI2, IC11G$1.PHI2, IC9G$1.PHI2
- net V33: no longer JP8.3
Other:
- note added: "1.1B: separate out PHI2_IO"
- note added: "MICROPET-V1.1B"
- note added: "MICROPET-V1.1B-20210122"
- note added: "MICROPET-V1.1B-20210622"
- note removed: "MICROPET-V1.0F-20210106"
- note removed: "MICROPET-V1.1A-20210601"
Changed lines of the file:
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@@
 <part name="V16" library="supply2" deviceset="VCC" device=""/>
 <part name="GND23" library="supply1" deviceset="GND" device=""/>
-<part name="JP8" library="jumper" deviceset="JP2E" device=""/>
 <part name="JP9" library="jumper" deviceset="JP2E" device=""/>
 <part name="GND24" library="supply1" deviceset="GND" device=""/>
@@
 <description>I/O</description>
 <plain>
-<text x="271.78" y="-93.98" size="2.54" layer="92">MICROPET-V1.1A-20210601</text>
-<text x="271.78" y="-71.12" size="3.81" layer="92">MICROPET-V1.1A</text>
+<text x="271.78" y="-93.98" size="2.54" layer="92">MICROPET-V1.1B-20210622</text>
+<text x="271.78" y="-71.12" size="3.81" layer="92">MICROPET-V1.1B</text>
 <text x="271.78" y="-76.2" size="2.54" layer="92">(C) A. Fachat</text>
 <text x="271.78" y="154.94" size="1.778" layer="91">Killer Poke Protection</text>
@@
 </segment>
 </net>
-<net name="PHI2" class="0">
+<net name="PHI2_IO" class="0">
 <segment>
 <wire x1="-99.06" y1="144.78" x2="-2.54" y2="144.78" width="0.1524" layer="91"/>
@@
 <description>RAM,ROM,CPU</description>
 <plain>
-<text x="271.78" y="0" size="2.54" layer="92">MICROPET-V1.0F-20210106</text>
-<text x="271.78" y="22.86" size="3.81" layer="92">MICROPET-V1.1A</text>
+<text x="271.78" y="0" size="2.54" layer="92">MICROPET-V1.1B-20210122</text>
+<text x="271.78" y="22.86" size="3.81" layer="92">MICROPET-V1.1B</text>
 <text x="271.78" y="17.78" size="2.54" layer="92">(C) A. Fachat</text>
 <text x="337.82" y="20.32" size="2.54" layer="92">SHEET 2/3</text>
@@
          (disables oscillators with Tri-state input)</text>
 <text x="279.4" y="60.96" size="2.54" layer="94">1.1A: replace parallel ROM with SPI Flash</text>
+<text x="279.4" y="66.04" size="2.54" layer="94">1.1B: separate out PHI2_IO</text>
 </plain>
 <instances>
@@
 <instance part="SUPPLY1" gate="G$1" x="-38.1" y="40.64"/>
 <instance part="GND20" gate="1" x="101.6" y="55.88"/>
-<instance part="JP8" gate="1" x="2.54" y="215.9" rot="R90"/>
 <instance part="JP9" gate="1" x="2.54" y="228.6" rot="R90"/>
 <instance part="GND24" gate="1" x="7.62" y="205.74"/>
@@
 <pinref part="GND24" gate="1" pin="GND"/>
 <wire x1="5.08" y1="226.06" x2="7.62" y2="226.06" width="0.1524" layer="91"/>
-<wire x1="7.62" y1="226.06" x2="7.62" y2="213.36" width="0.1524" layer="91"/>
-<pinref part="JP8" gate="1" pin="1"/>
-<wire x1="7.62" y1="213.36" x2="7.62" y2="208.28" width="0.1524" layer="91"/>
-<wire x1="5.08" y1="213.36" x2="7.62" y2="213.36" width="0.1524" layer="91"/>
-<junction x="7.62" y="213.36"/>
+<wire x1="7.62" y1="226.06" x2="7.62" y2="208.28" width="0.1524" layer="91"/>
 </segment>
 <segment>
@@
 </segment>
 <segment>
-<pinref part="JP8" gate="1" pin="3"/>
-<wire x1="5.08" y1="218.44" x2="10.16" y2="218.44" width="0.1524" layer="91"/>
-<wire x1="10.16" y1="218.44" x2="10.16" y2="231.14" width="0.1524" layer="91"/>
 <pinref part="JP9" gate="1" pin="3"/>
 <wire x1="5.08" y1="231.14" x2="10.16" y2="231.14" width="0.1524" layer="91"/>
-<junction x="10.16" y="231.14"/>
 <wire x1="10.16" y1="231.14" x2="10.16" y2="238.76" width="0.1524" layer="91"/>
 <wire x1="10.16" y1="238.76" x2="17.78" y2="238.76" width="0.1524" layer="91"/>
@@
 </segment>
 </net>
-<net name="PHI2" class="0">
-<segment>
-<pinref part="U$1" gate="G$1" pin="PH2-IN"/>
-<wire x1="66.04" y1="58.42" x2="55.88" y2="58.42" width="0.1524" layer="91"/>
-<wire x1="55.88" y1="58.42" x2="40.64" y2="58.42" width="0.1524" layer="91"/>
-<wire x1="40.64" y1="58.42" x2="40.64" y2="162.56" width="0.1524" layer="91"/>
-<pinref part="U$2" gate="G$3" pin="GTS0"/>
-<wire x1="40.64" y1="162.56" x2="124.46" y2="162.56" width="0.1524" layer="91"/>
-<wire x1="124.46" y1="162.56" x2="124.46" y2="170.18" width="0.1524" layer="91"/>
-<label x="48.26" y="58.42" size="1.27" layer="95"/>
-<label x="111.76" y="162.56" size="1.27" layer="95"/>
-<wire x1="40.64" y1="162.56" x2="20.32" y2="162.56" width="0.1524" layer="91"/>
-<junction x="40.64" y="162.56"/>
-<label x="22.86" y="162.56" size="1.27" layer="95"/>
-<pinref part="R12" gate="G$1" pin="2"/>
-<wire x1="55.88" y1="35.56" x2="55.88" y2="58.42" width="0.1524" layer="91"/>
-<junction x="55.88" y="58.42"/>
-</segment>
-</net>
 <net name="R/-W" class="0">
 <segment>
@@
 </segment>
 </net>
-<net name="MODE1" class="0">
+<net name="PHI2_IO" class="0">
 <segment>
-<pinref part="JP8" gate="1" pin="2"/>
-<wire x1="5.08" y1="215.9" x2="22.86" y2="215.9" width="0.1524" layer="91"/>
-<wire x1="22.86" y1="215.9" x2="22.86" y2="233.68" width="0.1524" layer="91"/>
 <pinref part="U$2" gate="G$3" pin="FB9MC14"/>
-<wire x1="22.86" y1="233.68" x2="132.08" y2="233.68" width="0.1524" layer="91"/>
+<wire x1="30.48" y1="233.68" x2="132.08" y2="233.68" width="0.1524" layer="91"/>
 <wire x1="132.08" y1="233.68" x2="132.08" y2="208.28" width="0.1524" layer="91"/>
 <label x="71.12" y="233.68" size="1.6764" layer="95"/>
 <label x="132.08" y="210.82" size="1.27" layer="95" rot="R90"/>
+<wire x1="20.32" y1="167.64" x2="30.48" y2="167.64" width="0.1524" layer="91"/>
+<wire x1="30.48" y1="167.64" x2="30.48" y2="233.68" width="0.1524" layer="91"/>
+<label x="22.86" y="167.64" size="1.27" layer="95"/>
 </segment>
 </net>
@@
 </segment>
 </net>
+<net name="PHI2" class="0">
+<segment>
+<pinref part="U$1" gate="G$1" pin="PH2-IN"/>
+<wire x1="66.04" y1="58.42" x2="55.88" y2="58.42" width="0.1524" layer="91"/>
+<wire x1="55.88" y1="58.42" x2="40.64" y2="58.42" width="0.1524" layer="91"/>
+<wire x1="40.64" y1="58.42" x2="40.64" y2="162.56" width="0.1524" layer="91"/>
+<pinref part="U$2" gate="G$3" pin="GTS0"/>
+<wire x1="40.64" y1="162.56" x2="124.46" y2="162.56" width="0.1524" layer="91"/>
+<wire x1="124.46" y1="162.56" x2="124.46" y2="170.18" width="0.1524" layer="91"/>
+<label x="48.26" y="58.42" size="1.27" layer="95"/>
+<label x="111.76" y="162.56" size="1.27" layer="95"/>
+<wire x1="40.64" y1="162.56" x2="20.32" y2="162.56" width="0.1524" layer="91"/>
+<junction x="40.64" y="162.56"/>
+<label x="22.86" y="162.56" size="1.27" layer="95"/>
+<pinref part="R12" gate="G$1" pin="2"/>
+<wire x1="55.88" y1="35.56" x2="55.88" y2="58.42" width="0.1524" layer="91"/>
+<junction x="55.88" y="58.42"/>
+</segment>
+</net>
