File: Board/micropet_v2.brd (EAGLE design)
At the start: 160.2 x 100.1 mm, 130 parts, among them CN3 PORT_CASSETTE_EDGE, CN4 PORT_IEEE_EDGE, IC1 RAMSOCK32TO512KSOP, IC10 PIAPLCC, IC11 PIAPLCC, IC13 RAMSOCK32TO512KSOP, IC2 74LS245DW, IC3 74HCT00D, IC4 74LS86D, IC5 74LS145N, IC8 MAX3421E, IC9 VIAPLCC, J1 DCJ0202, P1 C64KEYB, P2 IEEE488FLATCABLE, P3 PETUSERPORT, P6 CBMTAPE, P7 PETKEYBD, Q1 IRLML5203, Q2 32kHz, Q3 12MHz, X2 D-SUB15-HDR15RA

Commit message: update board to 2.0C
Parts:
- moved R9 0.16 mm to (54.3, 58.8)
Connections:
- new net FOO: U$12.3V3
- net V33: now also R9.1; no longer U$12.3V3
- net VCC: no longer R9.1
Routing:
- net V33: track 419.8 -> 463.9 mm, vias 17 -> 21
- net VCC: track 1099.3 -> 1090.4 mm
- net SPI_NSEL2: track 94.5 -> 97.5 mm, vias 8 -> 6
- net /IRQ: track 213.1 -> 214.4 mm
- net DENA: track 52.1 -> 51.2 mm
- net PHI2: track 55.6 -> 54.8 mm
- net D1: track 177.7 -> 178.4 mm
- net VSYNC: track 50.9 -> 50.3 mm
- net N$14: track 30.5 -> 31.0 mm
Other:
- board text added: "MicroPET-V2.0C"
- board text removed: "MicroPET-V2.0B"

Commit message: Micropet V2.1A
Parts:
- added C41, C42, C43, C44, C45, C46, C47, C48: 0.1u, rcl:C0603
- added JP6: (no value), jumper:JP2
- RN2, RN4: value 5k1 -> 2k4
- RN3, RN5: value 2k4 -> 5k1
- moved JP10 24.7 mm to (137.6, 73.7)
- moved C1 2.25 mm to (48.7, 40.9)
- moved C2 1.11 mm to (24.8, 39.5)
- moved C35 0.95 mm to (135.6, 76.8)
- moved C6 0.50 mm to (139.8, 79.5)
- moved IC4 0.08 mm to (140.0, 57.6)
Connections:
- net N$16 renamed REN
- new net ATNA_EN: IC3.10, IC3.5, JP10.2
- new net C2SW/ATNIN: IC10.8, JP6.2
- net /C1MTR: no longer IC3.12, IC3.13
- net /C2MTR: now also IC3.12, IC3.13
- net ATN: now also IC3.4
- net C2SW: now also JP6.1; no longer IC10.8
- net GND: now also C41.2, C42.2, C43.2, C44.2, C45.2, C46.2, C47.2, C48.2, JP10.3
- net N$11: now also U$6.6, U$6.7; no longer JP10.1
- net N$12: now also IC3.6, JP6.3; no longer IC3.10, IC3.11
- net N$2: now also IC3.11, JP10.1; no longer JP10.2, U$6.6, U$6.7
- net V33: now also C41.1, C42.1, C43.1, C44.1, C45.1, C46.1, C47.1, C48.1
- net VCC: no longer JP10.3
Routing:
- net /C2MTR: track 25.4 -> 130.4 mm, vias 2 -> 7
- net N$2: track 59.1 -> 8.18 mm, vias 3 -> 1
- net GND: track 1413.1 -> 1459.4 mm, vias 73 -> 78
- net N$11: track 32.0 -> 75.3 mm, vias 3 -> 4
- net /C1MTR: track 61.4 -> 27.5 mm, vias 3 -> 2
- net N$12: track 5.08 -> 27.4 mm, vias 0 -> 2
- net V33: track 463.9 -> 478.6 mm, vias 21 -> 23
- net C2SW/ATNIN: track 0.00 -> 13.5 mm, vias 0 -> 1
- net ATN: track 141.2 -> 152.6 mm
- net C2SW: track 96.8 -> 107.1 mm, vias 3 -> 5
- net ATNA_EN: track 0.00 -> 9.52 mm
- net N$1: track 23.7 -> 18.7 mm
- net VCC: track 1090.4 -> 1088.4 mm, vias 41 -> 42
- net N$44: track 97.3 -> 98.9 mm
- net DIO1: track 73.7 -> 74.9 mm
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Other:
- board text added: "MicroPET-V2.1A"
- board text removed: "MicroPET-V2.0C"
