File: Board/micropet_v2.sch (EAGLE design)
At the start: 130 parts, among them CN3 PORT_CASSETTE_EDGE, CN4 PORT_IEEE_EDGE, IC1 RAMSOCK32TO512KSOP, IC10 PIAPLCC, IC11 PIAPLCC, IC13 RAMSOCK32TO512KSOP, IC2 74LS245DW, IC3 74HCT00D, IC4 74LS86D, IC5 74LS145N, IC8 MAX3421E, IC9 VIAPLCC, J1 DCJ0202, P1 C64KEYB, P2 IEEE488FLATCABLE, P3 PETUSERPORT, P6 CBMTAPE, P7 PETKEYBD, Q1 IRLML5203, Q2 32kHz, Q3 12MHz, X2 D-SUB15-HDR15RA

Commit message: update board to 2.0C
Connections:
- new net FOO: U$12.V33
- net V33: now also R9.1
- net VCC: no longer R9.1
Other:
- note added: "MICROPET-V2.0C"
- note added: "MICROPET-V2.0C-20210515"
- note added: "V2.0B: - do not use '245 level converter but pullup R for PHI2 and PHI2_IO - Add missing SPI_NSEL5"
- note added: "V2.0B: do not use '245 level converter for PHI2 and PHI2_IO"
- note added: "V2.0C: pull up on /IRQ to 3.3V, to protect SPI devices from 5V"
- note removed: "MICROPET-V2.0A"
- note removed: "MICROPET-V2.0B"
- note removed: "Note: PHI2_IO_OUT and SPI_NSEL5 are unconnected on board!"
Changed lines of the file:
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@@
 <plain>
 <text x="325.12" y="-106.68" size="2.54" layer="92">MICROPET-V2.0A-20210130</text>
-<text x="325.12" y="-83.82" size="3.81" layer="92">MICROPET-V2.0A</text>
+<text x="325.12" y="-83.82" size="3.81" layer="92">MICROPET-V2.0C</text>
 <text x="325.12" y="-88.9" size="2.54" layer="92">(C) A. Fachat</text>
 <text x="147.32" y="127" size="1.778" layer="91">$E82x</text>
@@
 <description>CPU,RAM,ROM</description>
 <plain>
-<text x="271.78" y="0" size="2.54" layer="92">MICROPET-V2.0B-20210509</text>
-<text x="271.78" y="22.86" size="3.81" layer="92">MICROPET-V2.0B</text>
+<text x="271.78" y="0" size="2.54" layer="92">MICROPET-V2.0C-20210515</text>
+<text x="271.78" y="22.86" size="3.81" layer="92">MICROPET-V2.0C</text>
 <text x="271.78" y="17.78" size="2.54" layer="92">(C) A. Fachat</text>
 <text x="337.82" y="20.32" size="2.54" layer="92">SHEET 2/3</text>
-<text x="287.02" y="33.02" size="2.54" layer="94">Note: PHI2_IO_OUT and SPI_NSEL5
-         are unconnected on board!</text>
+<text x="271.78" y="45.72" size="2.54" layer="94">V2.0C: pull up on /IRQ to 3.3V, to protect SPI devices from 5V</text>
+<text x="271.78" y="33.02" size="2.54" layer="94">V2.0B: - do not use '245 level converter but pullup R
+              for PHI2 and PHI2_IO
+           - Add missing SPI_NSEL5</text>
 </plain>
 <instances>
@@
 <junction x="104.14" y="68.58"/>
 <junction x="104.14" y="20.32"/>
-<pinref part="R9" gate="G$1" pin="1"/>
-<wire x1="99.06" y1="20.32" x2="63.5" y2="20.32" width="0.1524" layer="91"/>
-<wire x1="63.5" y1="20.32" x2="63.5" y2="25.4" width="0.1524" layer="91"/>
+<wire x1="99.06" y1="20.32" x2="55.88" y2="20.32" width="0.1524" layer="91"/>
 <junction x="99.06" y="20.32"/>
 <pinref part="R12" gate="G$1" pin="1"/>
-<wire x1="63.5" y1="20.32" x2="55.88" y2="20.32" width="0.1524" layer="91"/>
 <wire x1="55.88" y1="20.32" x2="55.88" y2="25.4" width="0.1524" layer="91"/>
-<junction x="63.5" y="20.32"/>
 <label x="101.6" y="93.98" size="1.778" layer="95"/>
 </segment>
@@
 <label x="-43.18" y="246.38" size="1.27" layer="95"/>
 </segment>
+<segment>
+<pinref part="R9" gate="G$1" pin="1"/>
+<wire x1="63.5" y1="25.4" x2="63.5" y2="22.86" width="0.1524" layer="91"/>
+<wire x1="63.5" y1="22.86" x2="78.74" y2="22.86" width="0.1524" layer="91"/>
+<label x="71.12" y="22.86" size="1.27" layer="95"/>
+</segment>
 </net>
 <net name="/SEL1" class="0">
@@
 <plain>
 <text x="187.96" y="7.62" size="2.54" layer="92">MICROPET-V2.0A-20210130</text>
-<text x="187.96" y="30.48" size="3.81" layer="92">MICROPET-V2.0A</text>
+<text x="187.96" y="30.48" size="3.81" layer="92">MICROPET-V2.0C</text>
 <text x="187.96" y="25.4" size="2.54" layer="92">(C) A. Fachat</text>
 <wire x1="-2.54" y1="0" x2="287.02" y2="0" width="0.1524" layer="94"/>
@@
 <plain>
 <text x="190.5" y="7.62" size="2.54" layer="92">MICROPET-V2.0B-20210509</text>
-<text x="190.5" y="30.48" size="3.81" layer="92">MICROPET-V2.0B</text>
+<text x="190.5" y="30.48" size="3.81" layer="92">MICROPET-V2.0C</text>
 <text x="190.5" y="25.4" size="2.54" layer="92">(C) A. Fachat</text>
 <wire x1="0" y1="0" x2="289.56" y2="0" width="0.1524" layer="94"/>
@@
 <wire x1="0" y1="0" x2="0" y2="144.78" width="0.1524" layer="94"/>
 <wire x1="0" y1="144.78" x2="289.56" y2="144.78" width="0.1524" layer="94"/>
+<text x="187.96" y="38.1" size="2.54" layer="94">V2.0B: do not use '245 level converter for PHI2 and PHI2_IO</text>
 </plain>
 <instances>
@@
 <text x="25.4" y="63.5" size="1.778" layer="94">package layout by SparkFun</text>
 <text x="190.5" y="7.62" size="2.54" layer="92">MICROPET-V2.0A-20210306</text>
-<text x="190.5" y="30.48" size="3.81" layer="92">MICROPET-V2.0A</text>
+<text x="190.5" y="30.48" size="3.81" layer="92">MICROPET-V2.0C</text>
 <text x="190.5" y="25.4" size="2.54" layer="92">(C) A. Fachat</text>
 <wire x1="0" y1="0" x2="289.56" y2="0" width="0.1524" layer="94"/>
@@
 <pinref part="U$12" gate="G$1" pin="VIN"/>
 <pinref part="SUPPLY5" gate="G$1" pin="VCC"/>
-<wire x1="114.3" y1="134.62" x2="101.6" y2="134.62" width="0.1524" layer="91"/>
 <pinref part="C16" gate="G$1" pin="1"/>
+<wire x1="114.3" y1="134.62" x2="101.6" y2="134.62" width="0.1524" layer="91"/>
 <wire x1="101.6" y1="134.62" x2="99.06" y2="134.62" width="0.1524" layer="91"/>
 <wire x1="99.06" y1="132.08" x2="101.6" y2="132.08" width="0.1524" layer="91"/>
 <wire x1="101.6" y1="132.08" x2="101.6" y2="134.62" width="0.1524" layer="91"/>
 <junction x="101.6" y="134.62"/>
+<label x="104.14" y="134.62" size="1.778" layer="95"/>
 </segment>
 </net>
@@
 </segment>
 </net>
+<net name="FOO" class="0">
+<segment>
+<pinref part="U$12" gate="G$1" pin="V33"/>
+<wire x1="114.3" y1="132.08" x2="106.68" y2="132.08" width="0.1524" layer="91"/>
+</segment>
+</net>

Commit message: Micropet V2.1A
Parts:
- added C41, C42, C43, C44, C45, C46, C47, C48: 0.1u, rcl:C-EUC0603
- added JP6: (no value), jumper:JP2E
- RN2, RN4: value 5k1 -> 2k4
- RN3, RN5: value 2k4 -> 5k1
Connections:
- net N$16 renamed REN
- new net ATNA_EN: IC3B.I1, IC3C.I1, JP10.2
- new net C2SW/ATNIN: IC10G$1.PA5, JP6.2
- net /C1MTR: no longer IC3D.I0, IC3D.I1
- net /C2MTR: now also IC3D.I0, IC3D.I1
- net ATN: now also IC3B.I0
- net C2SW: now also JP6.1; no longer IC10G$1.PA5
- net GND: now also C41.2, C42.2, C43.2, C44.2, C45.2, C46.2, C47.2, C48.2, JP10.3
- net N$11: now also U$6G$1.A5, U$6G$1.A6; no longer JP10.1
- net N$12: now also IC3B.O, JP6.3; no longer IC3C.I1, IC3D.O
- net N$2: now also IC3D.O, JP10.1; no longer JP10.2, U$6G$1.A5, U$6G$1.A6
- net V33: now also C41.1, C42.1, C43.1, C44.1, C45.1, C46.1, C47.1, C48.1
- net VCC: no longer JP10.3
Other:
- note added: "Changes: 2.1A: align ATNA with CSA_PETIO_1.2A 5k1 pull down, 2k4 pull up for IEEE488 according to MC3446 datasheet."
- note added: "Changes: 2.1A: more bypass caps for CPLD"
- note added: "MICROPET-V2.1A"
- note added: "MICROPET-V2.1A-20211113"
- note added: "MICROPET-V2.1A-20220205"
- note added: "Optionally R18 = 2k4"
- note added: "SHEET 1/5"
- note added: "SHEET 2/5"
- note added: "SHEET 3/5"
- note added: "SHEET 4/5"
- note added: "V2.0B: do not use '245 level converter for PHI2 and PHI2_IO V2.1A: Value of R18 optionally as 2k4"
- note removed: "MICROPET-V2.0A-20210130"
- note removed: "MICROPET-V2.0B-20210509"
- note removed: "MICROPET-V2.0C"
- note removed: "SHEET 1/3"
- note removed: "SHEET 2/3"
- note removed: "SHEET 3/3"
- note removed: "SHEET 4/4"
- note removed: "V2.0B: do not use '245 level converter for PHI2 and PHI2_IO"
- moved on the sheet: IC3C, JP10, JP5, R3
